Commit message: feat: sync complete DR02 Pro model

File: robots/dr02_pro/urdf/DR02-pro.urdf (robot description, URDF)
Before this commit: robot DR02-pro, 32 links, 31 joints
Links:
- added link d435_front_link
- added link d435_head_link
- added link d435_rear_link
- added link imu_base_link
- added link imu_head_link
- added link left_hand_link, mass 0.230000; collision mesh filename=../meshes/left_hand_link.STL; visual mesh filename=../meshes/left_hand_link.STL
- added link lidar_link
- added link right_hand_link, mass 0.230000; collision mesh filename=../meshes/right_hand_link.STL; visual mesh filename=../meshes/right_hand_link.STL
- link base_link: geometry collision cylinder length=0.14 radius=0.085; visual mesh filename=../meshes/base_link.STL
- link body: geometry collision box size=0.2 0.23 0.11; collision box size=0.2 0.24 0.06
- link head_link: geometry collision sphere radius=0.115; visual mesh filename=../meshes/head_link.STL
- link left_ankle_x_link: geometry collision box size=0.3 0.11 0.06; visual mesh filename=../meshes/left_ankle_x_link.STL
- link left_ankle_y_link: geometry collision cylinder length=0.11 radius=0.044; visual mesh filename=../meshes/left_ankle_y_link.STL
- link left_elbow_link: geometry collision cylinder length=0.06 radius=0.045; collision cylinder length=0.11 radius=0.055
- link left_hip_x_link: geometry visual mesh filename=../meshes/left_hip_x_link.STL
- link left_hip_y_link: geometry collision cylinder length=0.135 radius=0.07; visual mesh filename=../meshes/left_hip_y_link.STL
- link left_hip_z_link: geometry collision cylinder length=0.22 radius=0.07; visual mesh filename=../meshes/left_hip_z_link.STL
- link left_knee_link: geometry collision cylinder length=0.14 radius=0.06; collision cylinder length=0.28 radius=0.06
- link left_shoulder_x_link: geometry collision cylinder length=0.055 radius=0.055; collision cylinder length=0.11 radius=0.055
- link left_shoulder_y_link: geometry visual mesh filename=../meshes/left_shoulder_y_link.STL
- link left_shoulder_z_link: geometry collision cylinder length=0.04 radius=0.057; visual mesh filename=../meshes/left_shoulder_z_link.STL
- link left_wrist_x_link: mass 0.388317 -> 0.158317; geometry visual mesh filename=../meshes/left_wrist_x_link.STL
- link left_wrist_y_link: geometry collision cylinder length=0.085 radius=0.035; visual mesh filename=../meshes/left_wrist_y_link.STL
- link left_wrist_z_link: geometry collision cylinder length=0.09 radius=0.042; visual mesh filename=../meshes/left_wrist_z_link.STL
- link neck_link: geometry collision cylinder length=0.07 radius=0.05; visual mesh filename=../meshes/neck_link.STL
- link right_ankle_x_link: geometry collision box size=0.3 0.11 0.06; visual mesh filename=../meshes/right_ankle_x_link.STL
- link right_ankle_y_link: geometry collision cylinder length=0.11 radius=0.044; visual mesh filename=../meshes/right_ankle_y_link.STL
- link right_elbow_link: geometry collision cylinder length=0.06 radius=0.045; collision cylinder length=0.11 radius=0.055
- link right_hip_x_link: geometry visual mesh filename=../meshes/right_hip_x_link.STL
- link right_hip_y_link: geometry collision cylinder length=0.135 radius=0.07; visual mesh filename=../meshes/right_hip_y_link.STL
- link right_hip_z_link: geometry collision cylinder length=0.22 radius=0.07; visual mesh filename=../meshes/right_hip_z_link.STL
- link right_knee_link: geometry collision cylinder length=0.14 radius=0.06; collision cylinder length=0.28 radius=0.06
- link right_shoulder_x_link: geometry collision cylinder length=0.055 radius=0.055; collision cylinder length=0.11 radius=0.055
- link right_shoulder_y_link: geometry visual mesh filename=../meshes/right_shoulder_y_link.STL
- link right_shoulder_z_link: geometry collision cylinder length=0.04 radius=0.057; visual mesh filename=../meshes/right_shoulder_z_link.STL
- link right_wrist_x_link: mass 0.388317 -> 0.158317; geometry visual mesh filename=../meshes/right_wrist_x_link.STL
- link right_wrist_y_link: geometry collision cylinder length=0.085 radius=0.035; visual mesh filename=../meshes/right_wrist_y_link.STL
- link right_wrist_z_link: geometry collision cylinder length=0.09 radius=0.042; visual mesh filename=../meshes/right_wrist_z_link.STL
- link waist_x_link: geometry collision box size=0.12 0.09 0.14; visual mesh filename=../meshes/waist_x_link.STL
- link waist_z_link: geometry collision cylinder length=0.04 radius=0.08; visual mesh filename=../meshes/waist_z_link.STL
Joints:
- added joint d435_front_joint: type fixed, parent body, child d435_front_link, origin xyz=0.12559 0.0175 0.078407 rpy=0 1.0472 0, axis 0 0 0
- added joint d435_head_joint: type fixed, parent body, child d435_head_link, origin xyz=0.11871 0.0175 0.5096 rpy=0 0.61086 0, axis 0 0 0
- added joint d435_rear_joint: type fixed, parent body, child d435_rear_link, origin xyz=-0.11241 -0.0175 -0.037264 rpy=0 1.0472 3.1416, axis 0 0 0
- added joint imu_base_joint: type fixed, parent body, child imu_base_link, origin xyz=-0.0003333 0.0014869 -0.3546 rpy=0 0 0, axis 0 0 0
- added joint imu_head_joint: type fixed, parent body, child imu_head_link, origin xyz=-0.0003333 0.021947 0.56429 rpy=0 0 0, axis 0 0 0
- added joint left_hand_joint: type fixed, parent left_wrist_x_link, child left_hand_link, origin xyz=0 0 -0.0602 rpy=0 0 0, axis 0 0 0
- added joint lidar_joint: type fixed, parent body, child lidar_link, origin xyz=0.09784 1.003E-05 0.4645 rpy=0 0 0, axis 0 0 0
- added joint right_hand_joint: type fixed, parent right_wrist_x_link, child right_hand_link, origin xyz=0 0 -0.0602 rpy=0 0 0, axis 0 0 0
- joint neck_y_joint: axis 0 1 0 -> (none); limit lower=-0.349066 upper=0.349066 effort=50 velocity=23.76 -> (none); type revolute -> fixed
- joint neck_z_joint: axis 0 0 1 -> (none); limit lower=-1.745329 upper=3.665191 effort=50 velocity=23.76 -> (none); type revolute -> fixed
